File: A1-External-ESP8266-Cooling-Fan-Module/A1-External-ESP8266-Cooling-Fan-Module.kicad_pcb (KiCad board)
At the start: 2 copper layers, 48 parts, among them J1 USB_B_Micro, J2 Fan connector, J3 Leds connector, Q1 SI2300, Q2 SI2300, Q3 SI2301, Q4 SI2301, Q5 SI2300, Q6 SI2300, U1 ESP12-F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

Commit message: final layout
Parts:
- added C10: 100n, Capacitor_SMD:C_0603_1608Metric, F.Cu at (237.6, 63.0)
- added C8: 100n, Capacitor_SMD:C_0603_1608Metric, F.Cu at (199.2, 67.8)
- added D10: LED, LED_SMD:LED_0805_2012Metric, F.Cu at (209.2, 50.6)
- added D4: LED, LED_SMD:LED_0805_2012Metric, F.Cu at (248.6, 75.4)
- added D5: LED, LED_SMD:LED_0805_2012Metric, F.Cu at (248.7, 69.9)
- added D6: LED, LED_SMD:LED_0805_2012Metric, F.Cu at (248.7, 64.7)
- added D7: LED, LED_SMD:LED_0805_2012Metric, F.Cu at (198.1, 72.8)
- added D8: LED, LED_SMD:LED_0805_2012Metric, F.Cu at (188.3, 69.3)
- added D9: LED, LED_SMD:LED_0805_2012Metric, F.Cu at (211.9, 52.2)
- added H1: MountingHole, MountingHole:MountingHole_3.2mm_M3_DIN965_Pad, F.Cu at (236.1, 46.3)
- added H2: MountingHole, MountingHole:MountingHole_3.2mm_M3_DIN965_Pad, F.Cu at (188.6, 75.3)
- added H3: MountingHole, MountingHole:MountingHole_3.2mm_M3_DIN965_Pad, F.Cu at (228.6, 96.3)
- added J4: PIR sensor, Connector_JST:JST_PH_B3B-PH-K_1x03_P2.00mm_Vertical, F.Cu at (243.0, 61.0)
- added J5: 24V IN, Connector_JST:JST_PH_B2B-PH-K_1x02_P2.00mm_Vertical, F.Cu at (243.0, 80.0)
- added J6: 3V3 OUT, Connector_JST:JST_PH_B2B-PH-K_1x02_P2.00mm_Vertical, F.Cu at (203.6, 95.0)
- added J7: LEDS, Connector_PinHeader_2.54mm:PinHeader_2x03_P2.54mm_Vertical, F.Cu at (243.5, 75.0)
- added J8: 3V3 OUT, Connector_JST:JST_PH_B2B-PH-K_1x02_P2.00mm_Vertical, F.Cu at (210.6, 95.0)
- added JP2: Cutoff bypass, Jumper:SolderJumper-2_P1.3mm_Open_RoundedPad1.0x1.5mm, F.Cu at (216.8, 70.3)
- added R20: 2k2, Resistor_SMD:R_0603_1608Metric, F.Cu at (246.5, 75.2)
- added R21: 130, Resistor_SMD:R_0603_1608Metric, F.Cu at (246.5, 69.7)
- added R22: 300, Resistor_SMD:R_0603_1608Metric, F.Cu at (246.5, 64.5)
- added R23: 0, Resistor_SMD:R_0603_1608Metric, F.Cu at (204.0, 44.5)
- added R24: 0, Resistor_SMD:R_0603_1608Metric, F.Cu at (205.3, 46.4)
- added R25: 0, Resistor_SMD:R_0603_1608Metric, F.Cu at (192.2, 67.7)
- added R26: 0, Resistor_SMD:R_0603_1608Metric, F.Cu at (194.1, 71.0)
- added R27: 0, Resistor_SMD:R_0603_1608Metric, F.Cu at (235.6, 63.0)
- C2: footprint Capacitor_SMD:C_1206_3216Metric -> Capacitor_SMD:CP_Elec_6.3x7.7
- C4: footprint Capacitor_THT:CP_Radial_D8.0mm_P3.80mm -> Capacitor_SMD:CP_Elec_8x10.5
- C5: footprint Capacitor_SMD:CP_Elec_6.3x7.7 -> Capacitor_SMD:CP_Elec_10x10.5
- R1, R18, R19, R2: value 4k7 -> 1k
- moved D1 184.0 mm to (229.9, 89.0), turned to 90 degrees
- moved U4 183.9 mm to (243.8, 91.6)
- moved R3 183.2 mm to (239.1, 98.8), turned to 180 degrees
- moved R4 178.6 mm to (234.9, 98.8), turned to 180 degrees
- moved C5 173.4 mm to (218.9, 80.0)
- moved C4 166.2 mm to (232.6, 80.0), turned to 180 degrees
- moved L1 146.0 mm to (219.0, 91.8), turned to 180 degrees
- moved R2 135.4 mm to (208.6, 46.4), turned to 90 degrees
- moved R1 133.5 mm to (212.3, 48.7), turned to 90 degrees
- moved C1 126.7 mm to (219.1, 55.0)
- moved D3 125.7 mm to (237.9, 55.0), turned to -90 degrees
- moved U5 121.4 mm to (231.1, 70.2), turned to -90 degrees
- moved C6 120.5 mm to (225.9, 67.4), turned to -90 degrees
- moved C7 120.1 mm to (225.9, 72.4), turned to 90 degrees
- moved J1 114.9 mm to (228.5, 45.0), turned to 180 degrees
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Connections:
- net Net-(Q3-S) renamed /LM2596-OUT
- Q2 pad 2: Net-(Q1-S) -> Net-(Q2-G)
- R1 pad 1: +3.3V -> Net-(D9-K)
- R12 pad 1: Net-(U3-~{RTS}) -> Net-(Q1-S)
- R12 pad 2: Net-(Q1-S) -> Net-(Q2-G)
- R18 pad 1: +3.3V -> Net-(D8-K)
- R18 pad 2: Net-(U1-GPIO5) -> Net-(U6-SCL)
- R19 pad 1: +3.3V -> Net-(D7-K)
- R19 pad 2: Net-(U1-GPIO4) -> Net-(U6-SDA)
- R2 pad 1: +3.3V -> Net-(D10-K)
- U1 pad 13: Net-(U1-GPIO4) -> ESP_PWM-FAN
- U1 pad 14: Net-(U1-GPIO5) -> ESP_PWM-LEDS
- U1 pad 15: ESP_RXD -> Net-(U1-RXD)
- U1 pad 16: ESP_TXD -> Net-(U1-TXD)
- U1 pad 6: ESP_PWM-LEDS -> /SCL
- U1 pad 7: ESP_PWM-FAN -> /SDA
- U3 pad 14: Net-(U3-~{RTS}) -> Net-(Q1-S)
- U6 pad 2: Net-(U1-GPIO4) -> Net-(U6-SDA)
- U6 pad 4: Net-(U1-GPIO5) -> Net-(U6-SCL)
Routing:
- net ESP_PIR-SENS: track 0.00 -> 54.0 mm, vias 0 -> 2
- net ESP_PWM-FAN: track 0.00 -> 44.1 mm, vias 0 -> 2
- net +5V: track 0.00 -> 39.8 mm
- net /LM2596-OUT: track 0.00 -> 38.8 mm
- net +3.3V: track 0.00 -> 38.2 mm, vias 0 -> 19
- net Net-(Q2-S): track 0.00 -> 35.2 mm, vias 0 -> 2
- net ESP_EN: track 0.00 -> 34.1 mm, vias 0 -> 2
- net ESP_GPIO0: track 6.02 -> 39.6 mm, vias 0 -> 2
- net ESP_PWM-LEDS: track 0.00 -> 32.6 mm, vias 0 -> 2
- net Net-(Q1-S): track 0.00 -> 32.2 mm
- net VBUS: track 3.25 -> 24.9 mm
- net ESP_TXD: track 0.00 -> 19.0 mm, vias 0 -> 2
- net ESP_RXD: track 0.00 -> 17.5 mm, vias 0 -> 2
- net Net-(J3-Pin_2): track 0.00 -> 16.4 mm
- net Net-(U6-SCL): track 0.00 -> 15.7 mm
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- added copper zone on F.Cu, net +24V
- added copper zone on In2.Cu, net +24V
- added copper zone on F.Cu, net +3.3V
- added copper zone on In2.Cu, net +3.3V
- added copper zone on F.Cu, net /LM2596-OUT
- added copper zone on F.Cu, net /OUT
- added copper zone on B.Cu, net GND
- added copper zone on F.Cu, net GND
- added copper zone on In1.Cu, net GND
Other:
- board outline added: 66 x 57 mm
- copper layers 2 -> 4
- board text added: "+"
- board text added: "-"
- board text added: "24V"
- board text added: "24V In"
- board text added: "3V3"
- board text added: "5V"
- board text added: "FAN"
- board text added: "GND"
- board text added: "LEDS"
- board text added: "PIR"
- board text added: "RX"
- board text added: "SCL"
- board text added: "SDA"
- board text added: "SENS"
- board text added: "TEMP/ HUM"
- board text added: "TX"
